Commit message: Update model.urdf.xacro
Add led plugin in urdf file

File: urdf/robobo/model.urdf.xacro (robot description, xacro)
@@ -343,4 +343,36 @@
 	</gazebo>
 </xacro:macro>
+<!--LEDs-->
+<xacro:macro name="LED" params="name xyz rpy">
+	<link name= "${name}">
+		<inertial>
+			<origin xyz="0 0 0" rpy="0 0 0"/>
+			<mass value="0.001" />
+			<inertia ixx="0.000001" ixy="0" ixz="0" iyy="0.000001" iyz="0" izz="0.000001"/>
+		</inertial>
+		<visual>
+			<origin xyz="0 0 0" rpy="0 0 0"/>
+			<geometry>
+				<cylinder radius="0.003" length="0.0005"/>
+			</geometry>
+		</visual>
+	</link>
+	<joint name="${name}" type="fixed">
+		<parent link="body" />
+		<child link="${name}"/>
+		<origin xyz="${xyz}" rpy="${rpy}"/>
+		<axis xyz="0 -1 0"/>
+	</joint>
+	<gazebo reference="${name}">
+		<visual>
+			<material>
+				<ambient>0 0 0 1</ambient>
+				<diffuse>0 0 0 1</diffuse>
+				<specular>0 0 0 0</specular>
+				<emissive>0 1 0 1</emissive>
+			</material>
+		</visual>
+	</gazebo>
+</xacro:macro>
 <!--PLUGINS OF MODEL-->
 <xacro:macro name="model_plugin">
@@ -373,4 +405,17 @@
 		</collision>
 	</link>
+	<!--LEDs-->
+	<xacro:LED name="Front-C" xyz="-0.0584 0 0.0328" rpy="0 -0.7 0"/>
+	<xacro:LED name="Front-R" xyz="-0.0709 0.0060 0.019" rpy="-0.09 -0.95 0"/>
+	<xacro:LED name="Front-RR" xyz="-0.0636	0.010	0.027" rpy="-0.15 -0.8 0"/>
+	<xacro:LED name="Front-L" xyz="-0.0709 -0.0060 0.019" rpy="0.09 -0.95 0"/>
+	<xacro:LED name="Front-LL" xyz="-0.0636 -0.010 0.027" rpy="0.15 -0.8 0"/>
+	<xacro:LED name="Back-L" xyz="0.084 -0.0372 0.02" rpy="1 0 0.35"/>
+	<xacro:LED name="Back-R" xyz="0.084 0.037 0.02" rpy="-1 0 -0.35"/>
+	<gazebo reference="Front-C">
+		<visual>
+			<plugin name="ledcolor_plugin" filename="libled_color.so"/>
+		</visual>
+	</gazebo>
 	<!--Use pusher-->
 	<xacro:if value="${pusher_xacro}">

Commit message: Update model.urdf.xacro

File: urdf/robobo/model.urdf.xacro (robot description, xacro)
@@ -25,5 +25,5 @@
 		<inertial>
 			<origin xyz="${0.01095+length/2} ${0.002} ${0.00215+depth/2}" rpy="0 0 0"/>
-			<mass value="${mass}"/>
+			<mass value="${mass/100}"/>
 			<inertia ixx="${mass*(width*width+depth*depth)/12}" ixy="0" ixz="0" iyy="${mass*(depth*depth+length*length)/12}" iyz="0" izz="${mass*(length*length+width*width)/12}"/>
 		</inertial>

Commit message: Update model.urdf.xacro

File: urdf/robobo/model.urdf.xacro (robot description, xacro)
@@ -25,5 +25,5 @@
 		<inertial>
 			<origin xyz="${0.01095+length/2} ${0.002} ${0.00215+depth/2}" rpy="0 0 0"/>
-			<mass value="${mass/100}"/>
+			<mass value="${mass}"/>
 			<inertia ixx="${mass*(width*width+depth*depth)/12}" ixy="0" ixz="0" iyy="${mass*(depth*depth+length*length)/12}" iyz="0" izz="${mass*(length*length+width*width)/12}"/>
 		</inertial>
@@ -389,5 +389,5 @@
 	<link name="body">
 		<inertial>
-			<origin xyz="0 0 0" rpy="0 0 0"/>
+			<origin xyz="0.04 0 0" rpy="0 0 0"/>
 			<mass value="0.6" />
 			<inertia ixx="0.000485229" ixy="0" ixz="0" iyy="0.001227181" iyz="0" izz="0.001452813"/>

Commit message: Update model.urdf.xacro

File: urdf/robobo/model.urdf.xacro (robot description, xacro)
@@ -25,5 +25,5 @@
 		<inertial>
 			<origin xyz="${0.01095+length/2} ${0.002} ${0.00215+depth/2}" rpy="0 0 0"/>
-			<mass value="${mass/100}"/>
+			<mass value="${mass}"/>
 			<inertia ixx="${mass*(width*width+depth*depth)/12}" ixy="0" ixz="0" iyy="${mass*(depth*depth+length*length)/12}" iyz="0" izz="${mass*(length*length+width*width)/12}"/>
 		</inertial>
@@ -388,5 +388,5 @@
 	<link name="body">
 		<inertial>
-			<origin xyz="0 0 0" rpy="0 0 0"/>
+			<origin xyz="0.04 0 0" rpy="0 0 0"/>
 			<mass value="0.6" />
 			<inertia ixx="0.000485229" ixy="0" ixz="0" iyy="0.001227181" iyz="0" izz="0.001452813"/>

Commit message: Update model.urdf.xacro

File: urdf/robobo/model.urdf.xacro (robot description, xacro)
@@ -25,5 +25,5 @@
 		<inertial>
 			<origin xyz="${0.01095+length/2} ${0.002} ${0.00215+depth/2}" rpy="0 0 0"/>
-			<mass value="${mass}"/>
+			<mass value="${mass/100}"/>
 			<inertia ixx="${mass*(width*width+depth*depth)/12}" ixy="0" ixz="0" iyy="${mass*(depth*depth+length*length)/12}" iyz="0" izz="${mass*(length*length+width*width)/12}"/>
 		</inertial>
@@ -104,4 +104,5 @@
 				</script>
 			</material>
+			<plugin name="emotion_plugin" filename="libemotion.so"/>
 		</visual>
 	</gazebo>
@@ -388,5 +389,5 @@
 	<link name="body">
 		<inertial>
-			<origin xyz="0.04 0 0" rpy="0 0 0"/>
+			<origin xyz="0 0 0" rpy="0 0 0"/>
 			<mass value="0.6" />
 			<inertia ixx="0.000485229" ixy="0" ixz="0" iyy="0.001227181" iyz="0" izz="0.001452813"/>
